Commit message: validate mjcf, update dyanamics notes

File: cara_description/urdf/cara_left_leg.urdf (robot description, URDF)
Before this commit: robot cara_left_leg, 7 links, 6 joints
Links:
- link l_foot: mass 0.05 -> 0.08
- link l_shin: mass 0.12 -> 0.18; geometry collision cylinder length=0.12 radius=0.018; visual cylinder length=0.12 radius=0.018
- link l_thigh: mass 0.15 -> 0.22; geometry collision cylinder length=0.12 radius=0.022; visual cylinder length=0.12 radius=0.022
- link pelvis: mass 0.6 -> 0.85
