Commit message: phase U2 complete

File: cara_description/urdf/cara_full_body.urdf (robot description, URDF)
Before this commit: robot cara_full_body, 14 links, 13 joints
Links:
- added link head, mass 0.35; collision sphere radius=0.06; visual sphere radius=0.06
- added link neck_roll_link
- added link neck_yaw_link
Joints:
- added joint neck_pitch: type fixed, parent neck_roll_link, child head, origin xyz=0 0 0 rpy=0 0 0
- added joint neck_roll: type fixed, parent neck_yaw_link, child neck_roll_link, origin xyz=0 0 0 rpy=0 0 0
- added joint neck_yaw: type fixed, parent torso, child neck_yaw_link, origin xyz=0 0 0.195 rpy=0 0 0

Commit message: phase U3 complete

File: cara_description/urdf/cara_full_body.urdf (robot description, URDF)
Before this commit: robot cara_full_body, 17 links, 16 joints
Links:
- added link battery, mass 0.25; collision box size=0.09 0.06 0.03; visual box size=0.09 0.06 0.03
- added link jetson, mass 0.15; collision box size=0.07 0.07 0.03; visual box size=0.07 0.07 0.03
Joints:
- added joint mount_battery: type fixed, parent pelvis, child battery, origin xyz=0 0 -0.03 rpy=0 0 0
- added joint mount_jetson: type fixed, parent pelvis, child jetson, origin xyz=0 0 -0.03 rpy=0 0 0

Commit message: phase U4 complete

File: cara_description/urdf/cara_full_body.urdf (robot description, URDF)
Before this commit: robot cara_full_body, 19 links, 18 joints
Links:
- added link l_arm, mass 0.18; collision cylinder length=0.19 radius=0.022; visual cylinder length=0.19 radius=0.022
- added link r_arm, mass 0.18; collision cylinder length=0.19 radius=0.022; visual cylinder length=0.19 radius=0.022
Joints:
- added joint l_shoulder: type fixed, parent torso, child l_arm, origin xyz=0 0.09 0.12 rpy=0 0 0
- added joint r_shoulder: type fixed, parent torso, child r_arm, origin xyz=0 -0.09 0.12 rpy=0 0 0

Commit message: phase U5 complete

File: cara_description/urdf/cara_full_body.urdf (robot description, URDF)
Before this commit: robot cara_full_body, 21 links, 20 joints
Links:
- added link l_ear, mass 0.02; collision box size=0.035 0.035 0.035; visual box size=0.035 0.035 0.035
- added link l_ear_servo, mass 0.01; collision box size=0.02 0.012 0.023; visual box size=0.02 0.012 0.023
- added link r_ear, mass 0.02; collision box size=0.035 0.035 0.035; visual box size=0.035 0.035 0.035
- added link r_ear_servo, mass 0.01; collision box size=0.02 0.012 0.023; visual box size=0.02 0.012 0.023
Joints:
- added joint l_ear_joint: type fixed, parent head, child l_ear, origin xyz=0.005 0.055 0.05 rpy=0 0 0
- added joint l_ear_servo_mount: type fixed, parent head, child l_ear_servo, origin xyz=0.005 0.03 0.045 rpy=0 0 0
- added joint r_ear_joint: type fixed, parent head, child r_ear, origin xyz=0.005 -0.055 0.05 rpy=0 0 0
- added joint r_ear_servo_mount: type fixed, parent head, child r_ear_servo, origin xyz=0.005 -0.03 0.045 rpy=0 0 0
